File: eaaeoe.kicad_sch (KiCad schematic)
At the start: 93 parts

Commit message: schematic = nicer
Other:
- note added: "Debug iface"
- note added: "PWR"
- note removed: "SYS PWR"
- moved on the sheet: C?, J?, U?E

Commit message: finish schematic, add cubemx project, some initial layout
Parts:
- removed C? (x2): 4.7u, Capacitor_SMD:C_0402_1005Metric, symbol Device:C_Small
- removed D? (x2): 1N5819WS, Diode_SMD:D_SOD-323, symbol Device:D_Schottky
- removed Q? (x4): MMBT2222A, Package_TO_SOT_SMD:SOT-23, symbol Device:Q_NPN_BEC
- removed Q? (x4): AO3400A, Package_TO_SOT_SMD:SOT-23, symbol Transistor_FET:AO3400A
- removed R?: 1k, Resistor_SMD:R_0603_1608Metric_Pad0.98x0.95mm_HandSolder, symbol Device:R_Small
- removed R? (x4): 5.1k, Resistor_SMD:R_0603_1608Metric_Pad0.98x0.95mm_HandSolder, symbol Device:R_Small
- added D2: LED_0603, LED_SMD:LED_0603_1608Metric_Pad1.05x0.95mm_HandSolder, symbol Device:LED
- added J5: AUDIO_HDR, Connector_PinSocket_2.54mm:PinSocket_2x03_P2.54mm_Vertical, symbol Connector_Generic:Conn_02x03_Odd_Even
- added J6: Conn_02x05_Odd_Even, Connector_PinHeader_2.54mm:PinHeader_2x05_P2.54mm_Vertical, symbol Connector_Generic:Conn_02x05_Odd_Even
- added Q1, Q2: S9015, Package_TO_SOT_SMD:SOT-23, symbol Device:Q_PNP_BEC
- added Q3, Q4, Q5, Q6: MMBT2222A, Package_TO_SOT_SMD:SOT-23, symbol Device:Q_NPN_BEC
- added R1, R7: 470, Resistor_SMD:R_0402_1005Metric, symbol Device:R_Small
- added R3, R4: 5.1k, Resistor_SMD:R_0402_1005Metric, symbol Device:R_Small
- added R5: 1k, Resistor_SMD:R_0402_1005Metric, symbol Device:R_Small
- C16, C18, C6, C7, C8, C9: renamed from C?; footprint Capacitor_SMD:C_0402_1005Metric -> Capacitor_THT:C_Disc_D10.0mm_W2.5mm_P5.00mm
- J1: renamed from J?; footprint (none) -> Connector_USB:USB_C_Receptacle_Amphenol_12401610E4-2A
- J2: renamed from J?; footprint (none) -> Connector_PinSocket_2.54mm:PinSocket_2x06_P2.54mm_Vertical
- J3: renamed from J?; footprint (none) -> Connector_Audio:Jack_3.5mm_CUI_SJ1-3535NG_Horizontal_CircularHoles
- J4: renamed from J?; footprint (none) -> Connector_RJ:RJ45_OST_PJ012-8P8CX_Vertical
- J7: renamed from J?; footprint (none) -> Connector_PinSocket_2.54mm:PinSocket_1x04_P2.54mm_Vertical
- L1: renamed from L?; footprint (none) -> Inductor_SMD:L_1206_3216Metric
- R10, R12, R13, R14, R15, R16, R17, R18, R19, R20, R21, R22, R23, R24, R25, R26, R27, R28, R29, R30, R31, R32, R33, R6, R9: renamed from R?; footprint Resistor_SMD:R_0603_1608Metric_Pad0.98x0.95mm_HandSolder -> Resistor_SMD:R_0402_1005Metric
- R2, R8: renamed from R?; value 1k -> 470; footprint Resistor_SMD:R_0603_1608Metric_Pad0.98x0.95mm_HandSolder -> Resistor_SMD:R_0402_1005Metric
- gave numbers to parts that had none: 33
Connections:
- net +5VA: now also J6.2 (Pin_2), Q1.2 (E), Q2.2 (E), R3.2, R4.2
- net AUDIO_CHL_PWM: now also J5.1 (Pin_1); no longer R15.2
- net AUDIO_CHR_PWM: now also J5.3 (Pin_3); no longer R23.2
- net CODEC_CK: now also J6.5 (Pin_5)
- net CODEC_SD: now also J6.9 (Pin_9)
- net CODEC_WS: now also J6.3 (Pin_3)
- net GND: now also J5.5 (Pin_5), J5.6 (Pin_6), J6.10 (Pin_10), J6.6 (Pin_6), Q3.2 (E), Q4.2 (E), Q5.2 (E), Q6.2 (E)
- net HBRG_O1: now also Q1.3 (C), Q5.3 (C)
- net HBRG_O2: now also Q2.3 (C), Q6.3 (C)
- net HBR_PWM_A: now also R5.2; no longer R6.2, R8.2
- net HBR_PWM_B: now also R6.2; no longer R2.2
- net PWR_O2: now also D2.1 (K)
- net VDD: now also J6.4 (Pin_4)
- net at D1.1 (K), R11.2: now also D2.2 (A)
- net at R6.1: now also Q4.1 (B)
- net CODEC_GPIO2: now reaches U4.29 (PB10)
- net CODEC_GPIO2: now also J6.8 (Pin_8)
- net CODEC_GPIO1: now reaches U4.30 (PB11)
- net CODEC_GPIO1: now also J6.1 (Pin_1)
- net CODEC_GPIO3: now reaches U4.35 (PB14)
- net CODEC_GPIO3: now also J6.7 (Pin_7)
- net at R2.1: now also Q2.1 (B)
- net at R8.1: now also Q6.1 (B)
- new net: Q3.1 (B), R5.1
- new net: Q5.1 (B), R7.1
- new net: Q3.3 (C), R1.2, R3.1, R7.2
- new net: J5.2 (Pin_2), R15.2
- new net: J5.4 (Pin_4), R23.2
- new net: Q1.1 (B), R1.1
- new net: Q4.3 (C), R2.2, R4.1, R8.2
Other:
- note added: "The amplitude should be the highest that's in linear range, so around 8V diff Based on https://www.ti.com/lit/an/sbaa265/sbaa265.pdf"
- note removed: "Charge pump for high side nmos"
- note removed: "Sth like 25khz"
- note removed: "The amplitude should be the highest that's in linear range, so around 8V diff"
- moved on the sheet: D1, R11, R2, R6, R8
